File: Hardware/HSM_Project.kicad_pcb (KiCad board)
At the start: 2 copper layers, 100.6 x 113.7 mm, 105 parts, among them J1 Conn_01x02_Pin, J10 VL530X Connector, J11 VL530X Connector, J12 VL530X Connector, J13 VL530X Connector, J14 BNO085 Breakout, J16 HC-05 Breakout Board, J2 MP1584 Breakout, J4 TEENSY_4.1, J5 Conn_01x08_Pin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

Commit message: Added KiCad backup files
Parts:
- moved Q9 0.55 mm to (177.0, 41.4)
- moved D1 0.12 mm to (137.5, 41.5)
- moved D9 0.12 mm to (108.1, 78.1)
Routing:
- net Net-(Q9-D): track 8.88 -> 7.47 mm
- net Net-(Q8-D): track 9.18 -> 8.18 mm
- net Net-(Q9-G): track 5.40 -> 5.93 mm
