File: Hardware/.history/Sensors.kicad_sch (KiCad schematic)
At the start: 57 parts, among them J10 VL530X Connector, J11 VL530X Connector, J12 VL530X Connector, J13 VL530X Connector, J14 BNO085 Breakout, J5 Conn_01x08_Pin, J8 VL530X Connector, J9 VL530X Connector, Q10 Q_NMOS_GSD, Q11 Q_NMOS_GSD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

Commit message: Updated the ootprint of emitter and reciver to pinheader, largened the logo
Parts:
- D1, D4, D6, D7, D8, D9: footprint SFH_4550:DIO_SFH_4550 -> Micromouse:SFH4550_HEADER
- Q13, Q3, Q4, Q5, Q6, Q7: footprint SFH_313_FA-3_4:XDCR_SFH_313_FA-3_4 -> Micromouse:SFH313_Header
Changed lines of the file:
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@@
 			)
 		)
-		(property "Footprint" "SFH_313_FA-3_4:XDCR_SFH_313_FA-3_4"
+		(property "Footprint" "Micromouse:SFH313_Header"
 			(at 152.4 97.79 0)
 			(hide yes)
@@
 			)
 		)
-		(property "Footprint" "SFH_4550:DIO_SFH_4550"
+		(property "Footprint" "Micromouse:SFH4550_HEADER"
 			(at 81.28 48.26 0)
 			(hide yes)
@@
 			)
 		)
-		(property "Footprint" "SFH_313_FA-3_4:XDCR_SFH_313_FA-3_4"
+		(property "Footprint" "Micromouse:SFH313_Header"
 			(at 78.74 97.79 0)
 			(hide yes)
@@
 			)
 		)
-		(property "Footprint" "SFH_313_FA-3_4:XDCR_SFH_313_FA-3_4"
+		(property "Footprint" "Micromouse:SFH313_Header"
 			(at 29.21 97.79 0)
 			(hide yes)
@@
 			)
 		)
-		(property "Footprint" "SFH_313_FA-3_4:XDCR_SFH_313_FA-3_4"
+		(property "Footprint" "Micromouse:SFH313_Header"
 			(at 102.87 97.79 0)
 			(hide yes)
@@
 			)
 		)
-		(property "Footprint" "SFH_313_FA-3_4:XDCR_SFH_313_FA-3_4"
+		(property "Footprint" "Micromouse:SFH313_Header"
 			(at 54.61 97.79 0)
 			(hide yes)
@@
 			)
 		)
-		(property "Footprint" "SFH_4550:DIO_SFH_4550"
+		(property "Footprint" "Micromouse:SFH4550_HEADER"
 			(at 156.21 46.99 0)
 			(hide yes)
@@
 			)
 		)
-		(property "Footprint" "SFH_4550:DIO_SFH_4550"
+		(property "Footprint" "Micromouse:SFH4550_HEADER"
 			(at 232.41 48.26 0)
 			(hide yes)
@@
 			)
 		)
-		(property "Footprint" "SFH_313_FA-3_4:XDCR_SFH_313_FA-3_4"
+		(property "Footprint" "Micromouse:SFH313_Header"
 			(at 125.73 97.79 0)
 			(hide yes)
@@
 			)
 		)
-		(property "Footprint" "SFH_4550:DIO_SFH_4550"
+		(property "Footprint" "Micromouse:SFH4550_HEADER"
 			(at 119.38 48.26 0)
 			(hide yes)
@@
 			)
 		)
-		(property "Footprint" "SFH_4550:DIO_SFH_4550"
+		(property "Footprint" "Micromouse:SFH4550_HEADER"
 			(at 40.64 48.26 0)
 			(hide yes)
@@
 			)
 		)
-		(property "Footprint" "SFH_4550:DIO_SFH_4550"
+		(property "Footprint" "Micromouse:SFH4550_HEADER"
 			(at 193.04 44.45 0)
 			(hide yes)
